File: hardware/hexdigit.kicad_pcb (KiCad board)
At the start: 2 copper layers, 7 parts, among them IC1 ATTINY1634-MU, P1 CONN_01X05, P2 CONN_01X05

Commit message: * Tweaks
Parts:
- added REF**: Measurement_Point_Square-SMD-Pad_Small, Measurement_Points:Measurement_Point_Square-SMD-Pad_Small, F.Cu at (169.5, 102.9)
- added REF**: Measurement_Point_Round-SMD-Pad_Small, Measurement_Points:Measurement_Point_Round-SMD-Pad_Small, F.Cu at (167.8, 102.9)
- added REF**: Measurement_Point_Round-SMD-Pad_Small, Measurement_Points:Measurement_Point_Round-SMD-Pad_Small, F.Cu at (165.9, 102.9)
Routing:
- net Net-(AFF1-Pad5): track 15.9 -> 12.3 mm, vias 0 -> 2
- net Net-(AFF1-Pad4): track 10.8 -> 10.2 mm
